File: ZYNQ_PL.kicad_sch (KiCad schematic)
At the start: 17 parts, among them J6 BWSMA-KE-P001, J7 Conn_02x40_Odd_Even, U8 XC7Z020-CLG484

Commit message: 变压器输入+两块DDR3
Changed lines of the file:
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@@
       (effects (font (size 1.27 1.27)) hide)
     )
-    (property "Datasheet" "datasheet/X0511FVS-80A-LPV01_母.pdf" (at 138.43 87.63 0)
+    (property "Datasheet" "~" (at 138.43 87.63 0)
       (effects (font (size 1.27 1.27)) hide)
     )
@@
     )
     (property "Value" "BWSMA-KE-P001" (at 107.95 181.61 0)
-      (effects (font (size 1.27 1.27)))
+      (effects (font (size 1.27 1.27)) hide)
     )
     (property "Footprint" "footprints:SMA_Connect" (at 107.95 181.61 0)

Commit message: 删除-5V电源，添加eMMC模块接口
Parts:
- removed J7: Conn_02x40_Odd_Even, footprints:PinHeader_2x40_P0.5mm_Vertical_SMD, symbol Connector_Generic:Conn_02x40_Odd_Even
- added J11, J7: M50-490, Connector_PinHeader_1.27mm:PinHeader_2x10_P1.27mm_Vertical_SMD, symbol Connector_Generic:Conn_02x10_Odd_Even
- renumbered C163 to C159, C164 to C160, C165 to C161, C166 to C162, C167 to C163, C168 to C164, R54 to R33, R53 to R34, R55 to R35, R56 to R36, R57 to R37, R58 to R38
Connections:
- net Earth: now also J7.10 (Pin_10), J7.14 (Pin_14), J7.19 (Pin_19), J7.20 (Pin_20)
- net PL14_IO10_N: now also J11.11 (Pin_11)
- net PL14_IO10_P: now also J11.9 (Pin_9)
- net PL14_IO11_N: now also U8.AA19 (IO_L11N_T1_SRCC_33), J11.15 (Pin_15); no longer U8.U16 (IO_L15N_T2_DQS_33)
- net PL14_IO11_P: now also U8.Y19 (IO_L11P_T1_SRCC_33), J11.13 (Pin_13); no longer U8.U15 (IO_L15P_T2_DQS_33)
- net PL14_IO12_N: now also U8.AA18 (IO_L12N_T1_MRCC_33), J11.19 (Pin_19); no longer U8.V17 (IO_L16N_T2_33)
- net PL14_IO12_P: now also U8.Y18 (IO_L12P_T1_MRCC_33), J11.17 (Pin_17); no longer U8.U17 (IO_L16P_T2_33)
- net PL14_IO13_N: now also U8.W18 (IO_L13N_T2_MRCC_33), J11.4 (Pin_4); no longer U8.AB17 (IO_L17N_T2_33)
- net PL14_IO13_P: now also U8.W17 (IO_L13P_T2_MRCC_33), J11.2 (Pin_2); no longer U8.AA17 (IO_L17P_T2_33)
- net PL14_IO14_N: now also U8.Y16 (IO_L14N_T2_SRCC_33), J11.8 (Pin_8); no longer U8.AB16 (IO_L18N_T2_33)
- net PL14_IO14_P: now also U8.W16 (IO_L14P_T2_SRCC_33), J11.6 (Pin_6); no longer U8.AA16 (IO_L18P_T2_33)
- net PL14_IO15_N: now also U8.U16 (IO_L15N_T2_DQS_33), J11.12 (Pin_12); no longer U8.V15 (IO_L19N_T3_VREF_33)
- net PL14_IO15_P: now also U8.U15 (IO_L15P_T2_DQS_33), J11.10 (Pin_10); no longer U8.V14 (IO_L19P_T3_33)
- net PL14_IO16_N: now also U8.V17 (IO_L16N_T2_33), J11.16 (Pin_16); no longer U8.W13 (IO_L20N_T3_33)
- net PL14_IO16_P: now also U8.U17 (IO_L16P_T2_33), J11.14 (Pin_14); no longer U8.V13 (IO_L20P_T3_33)
- net PL14_IO17_N: now also U8.AB17 (IO_L17N_T2_33), J11.20 (Pin_20); no longer U8.Y15 (IO_L21N_T3_DQS_33)
- net PL14_IO17_P: now also U8.AA17 (IO_L17P_T2_33), J11.18 (Pin_18); no longer U8.W15 (IO_L21P_T3_DQS_33)
- net PL14_IO8_N: now also J11.3 (Pin_3)
- net PL14_IO8_P: now also J11.1 (Pin_1)
- net PL14_IO9_N: now also J11.7 (Pin_7)
- net PL14_IO9_P: now also J11.5 (Pin_5)
- net VCC_3V3: now also J7.18 (Pin_18)
- net eMMC_CMD: now reaches U8.AA6 (IO_L14N_T2_SRCC_13)
- net eMMC_CMD: now also J7.11 (Pin_11)
- net eMMC_RST: now reaches U8.AA7 (IO_L14P_T2_SRCC_13)
- net eMMC_RST: now also J7.17 (Pin_17)
- net eMMC_DS: now reaches U8.Y5 (IO_L13N_T2_MRCC_13)
- net eMMC_DS: now also J7.9 (Pin_9)
- net eMMC_CLK: now reaches U8.Y6 (IO_L13P_T2_MRCC_13)
- net eMMC_CLK: now also J7.12 (Pin_12)
- net PL13_IO10_N: no longer names the net of U8.Y10 (IO_L10N_T1_13)
- net PL13_IO10_P: no longer names the net of U8.Y11 (IO_L10P_T1_13)
- net PL13_IO11_N renamed eMMC_D1
- net eMMC_D1: now also J7.2 (Pin_2)
- net PL13_IO11_P renamed eMMC_D0
- net eMMC_D0: now also J7.1 (Pin_1)
- net PL13_IO12_N renamed eMMC_D3
- net eMMC_D3: now also J7.4 (Pin_4)
- net PL13_IO12_P renamed eMMC_D2
- net eMMC_D2: now also J7.3 (Pin_3)
- net PL13_IO13_N renamed eMMC_D5
- net eMMC_D5: now also J7.6 (Pin_6)
- net PL13_IO13_P renamed eMMC_D4
- net eMMC_D4: now also J7.5 (Pin_5)
- net PL13_IO14_N renamed eMMC_D7
- net eMMC_D7: now also J7.8 (Pin_8)
- net PL13_IO14_P renamed eMMC_D6
- net eMMC_D6: now also J7.7 (Pin_7)
- net PL13_IO15_N: no longer names the net of U8.T6 (IO_L19N_T3_VREF_13)
- net PL13_IO15_P: no longer names the net of U8.R6 (IO_L19P_T3_13)
- net PL13_IO16_N: no longer names the net of U8.U4 (IO_L20N_T3_13)
- net PL13_IO16_P: no longer names the net of U8.T4 (IO_L20P_T3_13)
- net PL13_IO17_N: no longer names the net of U8.V4 (IO_L21N_T3_DQS_13)
- net PL13_IO17_P: no longer names the net of U8.V5 (IO_L21P_T3_DQS_13)
- net PL13_IO18_N: no longer names the net of U8.U5 (IO_L22N_T3_13)
- net PL13_IO18_P: no longer names the net of U8.U6 (IO_L22P_T3_13)
- net PL13_IO19_N: no longer names the net of U8.W7 (IO_L23N_T3_13)
- net PL13_IO19_P: no longer names the net of U8.V7 (IO_L23P_T3_13)
- net PL13_IO1_N: no longer names the net of U8.V9 (IO_L1N_T0_13)
- net PL13_IO1_P: no longer names the net of U8.V10 (IO_L1P_T0_13)
- net PL13_IO20_N: no longer names the net of U8.W5 (IO_L24N_T3_13)
- net PL13_IO20_P: no longer names the net of U8.W6 (IO_L24P_T3_13)
- net PL13_IO2_N: no longer names the net of U8.W8 (IO_L2N_T0_13)
- net PL13_IO2_P: no longer names the net of U8.V8 (IO_L2P_T0_13)
- net PL13_IO3_N: no longer names the net of U8.W10 (IO_L3N_T0_DQS_13)
- net PL13_IO3_P: no longer names the net of U8.W11 (IO_L3P_T0_DQS_13)
- net PL13_IO4_N: no longer names the net of U8.W12 (IO_L4N_T0_13)
- net PL13_IO4_P: no longer names the net of U8.V12 (IO_L4P_T0_13)
- net PL13_IO5_N: no longer names the net of U8.U11 (IO_L5N_T0_13)
- net PL13_IO5_P: no longer names the net of U8.U12 (IO_L5P_T0_13)
- net PL13_IO6_N: no longer names the net of U8.U9 (IO_L6N_T0_VREF_13)
- net PL13_IO6_P: no longer names the net of U8.U10 (IO_L6P_T0_13)
- net PL13_IO7_N: no longer names the net of U8.AB12 (IO_L7N_T1_13)
- net PL13_IO7_P: no longer names the net of U8.AA12 (IO_L7P_T1_13)
- net PL13_IO8_N: no longer names the net of U8.AB11 (IO_L8N_T1_13)
- net PL13_IO8_P: no longer names the net of U8.AA11 (IO_L8P_T1_13)
- net PL13_IO9_N: no longer names the net of U8.AB9 (IO_L9N_T1_DQS_13)
- net PL13_IO9_P: no longer names the net of U8.AB10 (IO_L9P_T1_DQS_13)
- net PL14_IO18_N: no longer names the net of U8.AA14 (IO_L22N_T3_33)
- net PL14_IO18_P: no longer names the net of U8.Y14 (IO_L22P_T3_33)
- net PL14_IO19_N: no longer names the net of U8.AA13 (IO_L23N_T3_33)
- net PL14_IO19_P: no longer names the net of U8.Y13 (IO_L23P_T3_33)
- net PL14_IO1_N: no longer names the net of U8.U21 (IO_L1N_T0_33)
- net PL14_IO1_P: no longer names the net of U8.T21 (IO_L1P_T0_33)
- net PL14_IO20_N: no longer names the net of U8.AB15 (IO_L24N_T3_33)
- net PL14_IO20_P: no longer names the net of U8.AB14 (IO_L24P_T3_33)
- net PL14_IO2_N: no longer names the net of U8.U22 (IO_L2N_T0_33)
- net PL14_IO2_P: no longer names the net of U8.T22 (IO_L2P_T0_33)
- net PL14_IO3_N: no longer names the net of U8.W22 (IO_L3N_T0_DQS_33)
- net PL14_IO3_P: no longer names the net of U8.V22 (IO_L3P_T0_DQS_33)
- net PL14_IO4_N: no longer names the net of U8.W21 (IO_L4N_T0_33)
- net PL14_IO4_P: no longer names the net of U8.W20 (IO_L4P_T0_33)
- net PL14_IO5_N: no longer names the net of U8.V20 (IO_L5N_T0_33)
- net PL14_IO5_P: no longer names the net of U8.U20 (IO_L5P_T0_33)
- net PL14_IO6_N: no longer names the net of U8.V19 (IO_L6N_T0_VREF_33)
- net PL14_IO6_P: no longer names the net of U8.V18 (IO_L6P_T0_33)
- net PL14_IO7_N: no longer names the net of U8.AB22 (IO_L7N_T1_33)
- net PL14_IO7_P: no longer names the net of U8.AA22 (IO_L7P_T1_33)
- new net VCC_1V8: J7.16 (Pin_16)
- no-connect marks 58 -> 108
Other:
- note added: "PL Bank 13&33"
- note added: "PL Extension Connector"
- note added: "eMMC Module Connector"
- note removed: "PL Bank 13&33: Reserved"
- moved on the sheet: U8B, U8C
