File: ZYNQ_SD_ETH.kicad_sch (KiCad schematic)
At the start: 58 parts, among them J8 Micro_SD_Card_Det1, J9 HR911130A, U19 TXS02612RTW, U20 RTL8211F-CG, U8 XC7Z020-CLG484, Y1 25Mhz

Commit message: 变压器输入+两块DDR3
Parts:
- J9: footprint footprints:HR911130A -> HR911130A_HAN
- U20: footprint Package_DFN_QFN:QFN-40-1EP_5x5mm_P0.4mm_EP3.6x3.6mm -> RTL8211F-CG_RTK
Changed lines of the file:
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@@
       (effects (font (size 1.524 1.524)))
     )
-    (property "Footprint" "footprints:HR911130A" (at 218.44 166.37 0)
+    (property "Footprint" "HR911130A_HAN" (at 218.44 166.37 0)
       (effects (font (size 1.27 1.27) italic) hide)
     )
-    (property "Datasheet" "datasheet/HR911130A.pdf" (at 218.44 163.83 0)
+    (property "Datasheet" "HR911130A" (at 218.44 163.83 0)
       (effects (font (size 1.27 1.27) italic) hide)
     )
@@
       (effects (font (size 1.524 1.524)))
     )
-    (property "Footprint" "Package_DFN_QFN:QFN-40-1EP_5x5mm_P0.4mm_EP3.6x3.6mm" (at 175.26 81.28 0)
+    (property "Footprint" "RTL8211F-CG_RTK" (at 175.26 81.28 0)
       (effects (font (size 1.27 1.27) italic) hide)
     )
-    (property "Datasheet" "datasheet/RTL8211F-CG.PDF" (at 175.26 83.82 0)
+    (property "Datasheet" "RTL8211F-CG" (at 175.26 83.82 0)
       (effects (font (size 1.27 1.27) italic) hide)
     )
@@
       (effects (font (size 1.27 1.27)) hide)
     )
-    (property "Datasheet" "datasheet/X322525MOB4SI.pdf" (at 254 38.1 0)
-      (effects (font (size 1.27 1.27)) hide)
-    )
+    (property "Datasheet" "~" (at 254 38.1 0)
+      (effects (font (size 1.27 1.27)) hide)
+    )

Commit message: 删除-5V电源，添加eMMC模块接口
Parts:
- J9: footprint HR911130A_HAN -> footprints:HR911130A
- U12: renamed from U20; footprint RTL8211F-CG_RTK -> Package_DFN_QFN:QFN-40-1EP_5x5mm_P0.4mm_EP3.6x3.6mm
- renumbered C169 to C165, C170 to C166, C171 to C167, C172 to C168, C173 to C169, C174 to C170, C175 to C171, C176 to C172, C177 to C173, C178 to C174, C179 to C175, C180 to C176, C181 to C177, C182 to C178, C183 to C179, C184 to C180, C185 to C181, C186 to C182, C187 to C183, C188 to C184, C189 to C185, R59 to R39, R60 to R40, R61 to R41, R62 to R42, R63 to R43, R64 to R44, R65 to R45, R66 to R46, R67 to R47, R68 to R48, R69 to R49, R70 to R50, R71 to R51, R72 to R52, R73 to R53, R74 to R54, R75 to R55, R76 to R56, R77 to R57, R78 to R58, R79 to R59, R80 to R60, R81 to R61, R82 to R62, R83 to R63, R84 to R64, R85 to R65, U19 to U11
